File: pcb/pcb_v1.0/fpga.sch (KiCad schematic (older format))
At the start: 55 parts, among them P1 JTAG_CONN, U10 S25FL116K, U12 TLV70012, U13 TLV70025, U14 TLV70012, U2 EP4CE15E22

Commit message: Reordered inputs, improved clock layout
Connections:
- net labels added: CLK0
Other:
- moved on the sheet: R18
