File: pcb/pcb_v1.0/input1.sch (KiCad schematic (older format))
At the start: 26 parts

Commit message: Reordered inputs, improved clock layout
Parts:
- added C15, C9: 0.1u, custom_components:SM0603_Capa_libcms, symbol C
- added R4: 4.7k, custom_components:SM0603_Resistor_libcms, symbol R
- U6: renamed from U?; footprint (none) -> Housings_DFN_QFN:QFN-20-1EP_4x4mm_Pitch0.5mm
- gave numbers to parts that had none: 25
Connections:
- net IOVDD is gone; now on net VCCIO: C14.1, C6.2, C7.2, C8.2, U3.1 (A->B), U3.20 (VCC), U4.1 (A->B), U4.20 (VCC), U5.1 (A->B), U5.20 (VCC), U9.8 (Vcc)
- net B0_O: now also U4.11 (B7); no longer U4.18 (B0)
- net B1_O: now also U4.12 (B6); no longer U4.17 (B1)
- net B2_O: now also U4.13 (B5); no longer U4.16 (B2)
- net B3_O: now also U4.14 (B4); no longer U4.15 (B3)
- net F0_O: now also U3.15 (B3); no longer U4.14 (B4)
- net F1_O: now also U3.16 (B2); no longer U4.13 (B5)
- net F2_O: now also U3.17 (B1); no longer U4.12 (B6)
- net F3_O: now also U3.18 (B0); no longer U4.11 (B7)
- net G0_O: now also U4.15 (B3); no longer U3.14 (B4)
- net G1_O: now also U4.16 (B2); no longer U3.13 (B5)
- net G2_O: now also U4.17 (B1); no longer U3.12 (B6)
- net G3_O: now also U4.18 (B0); no longer U3.11 (B7)
- net GND: now also C15.1, C9.1
- net R0_O: now also U3.11 (B7); no longer U3.18 (B0)
- net R1_O: now also U3.12 (B6); no longer U3.17 (B1)
- net R2_O: now also U3.13 (B5); no longer U3.16 (B2)
- net R3_O: now also U3.14 (B4); no longer U3.15 (B3)
- net PCLKx2: now reaches U6.6 (CLKIN), U9.2 (3Y)
- net at U3.7 (A5): now also J2.4 (Pin_4); no longer J2.2 (Pin_2)
- net at U3.9 (A7): now also J2.2 (Pin_2); no longer J2.4 (Pin_4)
- net at U4.7 (A5): now also J1.4 (Pin_4); no longer J1.2 (Pin_2)
- net at U4.9 (A7): now also J1.2 (Pin_2); no longer J1.4 (Pin_4)
- net VCCIO: now reaches U6.10 (VDDOB)
- net VCCIO: now also U6.11 (VDDOA), U6.14 (VDDOD), U6.18 (VDDOC), U6.20 (VDD), C15.2, C9.2, R4.1
- net CLK0: now reaches U6.13 (CLK0)
- net at U6.3 (INTR#): now also R4.2
- no-connect marks 10 -> 17
Other:
- moved on the sheet: U6

Commit message: fix schematic and library linkage issues
Parts:
- D1: symbol ZENERsmall -> D_Zener_Small_ALT
- U6: footprint Housings_DFN_QFN:QFN-20-1EP_4x4mm_Pitch0.5mm -> custom_components:QFN-20-1EP_4x4mm_Pitch0.5mm_Handsoldering; symbol SI5351C-B -> Si5351C
