File: pcb/cps2_digiav.kicad_pcb (KiCad board)
At the start: 2 copper layers, 103.4 x 48.7 mm, 128 parts, among them J1 Conn_02x05, J2 Conn_02x05, J4 HDMI_CONN, P1 JTAG_CONN, U1 ADV7513, U10 IS25LP016D-JBLE, U12 TLV70012, U13 TLV70025, U14 TLV70012, U15 TLV70018, U16 TLV70018, U2 EP4CE15E22, U3 74LVC245, U4 74LVC245, U5 74LVC245, U6 SI5351C-B, U7 AP7361, U8 TLV70033, U9 SN74LVC3G17

Commit message: finalize schematic and do initial placement on PCB
Parts:
- added C16: 0.1u, custom_components:SM0603_Capa_libcms, F.Cu at (90.8, 80.1)
- added C17: 0.1u, custom_components:SM0603_Capa_libcms, F.Cu at (90.8, 84.4)
- added C18: 0.1u, custom_components:SM0603_Capa_libcms, F.Cu at (90.7, 78.1)
- added C19: 0.1u, custom_components:SM0603_Capa_libcms, F.Cu at (90.9, 86.1)
- added C20: 0.1u, custom_components:SM0603_Capa_libcms, F.Cu at (91.0, 87.9)
- added C21: 0.1u, custom_components:SM0603_Capa_libcms, F.Cu at (91.0, 89.9)
- added C22: 0.1u, custom_components:SM0603_Capa_libcms, F.Cu at (91.1, 91.9)
- added C23: 0.1u, custom_components:SM0603_Capa_libcms, F.Cu at (91.2, 96.4)
- added C24: 10u, custom_components:SM0603_Capa_libcms, F.Cu at (91.1, 98.4)
- added C25: 0.1u, custom_components:SM0603_Capa_libcms, F.Cu at (91.3, 100.6)
- added C26: 10u, custom_components:SM0603_Capa_libcms, F.Cu at (90.8, 82.3)
- added J3: GS2, Connectors:GS2, F.Cu at (74.2, 76.6)
- added J5: GS2, Connectors:GS2, F.Cu at (76.5, 76.7)
- added J6: GS2, Connectors:GS2, F.Cu at (79.0, 76.6)
- added R5: 2.2k, custom_components:SM0603_Resistor_libcms, F.Cu at (91.1, 94.3)
- added U11: SRC4190, Housings_SSOP:SSOP-28_5.3x10.2mm_Pitch0.65mm, F.Cu at (76.3, 66.5)
- R41: value 4.7k -> 10k
- R45, R46: value 4.7k -> 2.2k
- U1: footprint Housings_QFP:LQFP-64-1EP_10x10mm_Pitch0.5mm -> custom_components:LQFP-64-1EP_10x10mm_Pitch0.5mm_Handsoldering
- U2: value EP4CE15E22 -> 10CL025YE144C8N
- moved W2 36.7 mm to (45.5, 70.4), turned to 90 degrees
- moved W3 35.2 mm to (47.4, 70.4), turned to 90 degrees
- moved W4 33.7 mm to (49.3, 70.4), turned to 90 degrees
- moved W5 32.4 mm to (51.2, 70.4), turned to 90 degrees
- moved U5 31.6 mm to (64.2, 68.5)
- moved W6 31.3 mm to (53.1, 70.4), turned to 90 degrees
- moved U10 26.3 mm to (64.2, 29.3), turned to 0 degrees
- moved P1 21.4 mm to (46.8, 37.7), turned to 270 degrees
- moved U3 17.9 mm to (64.2, 38.3)
- moved R3 6.53 mm to (126.1, 46.4)
- moved C94 3.14 mm to (81.7, 63.6)
- moved R4 3.11 mm to (81.7, 65.4)
- moved U1 3.00 mm to (117.8, 36.0)
- turned U2 to 90 degrees
Connections:
- U1 pad 22: /fpga1/HDMITX_RESET_N -> GND
- U1 pad 3: Net-(U1-Pad3) -> GND
- U1 pad 32: Net-(U1-Pad32) -> GND
- U1 pad 4: /fpga1/AUD_MCLK -> GND
- U1 pad 6: Net-(U1-Pad6) -> GND
- U1 pad 7: Net-(U1-Pad7) -> GND
- U1 pad 8: Net-(U1-Pad8) -> GND
- U2 pad 10: /fpga1/HDMITX_R6 -> /fpga1/SDOUT
- U2 pad 100: /fpga1/AUD_MCLK -> /fpga1/HDMITX_R4
- U2 pad 101: /fpga1/HDMITX_VSYNC -> /fpga1/HDMITX_R5
- U2 pad 103: /fpga1/HDMITX_HSYNC -> /fpga1/HDMITX_R6
- U2 pad 104: /hdmitx1/DE -> GND
- U2 pad 105: /hdmitx1/B0 -> Net-(U2-Pad105)
- U2 pad 106: /hdmitx1/B1 -> /fpga1/HDMITX_R7
- U2 pad 11: /fpga1/HDMITX_R7 -> /fpga1/LRCKO
- U2 pad 110: /hdmitx1/B2 -> GND
- U2 pad 111: /hdmitx1/B3 -> /input1/F3_O
- U2 pad 112: /hdmitx1/B4 -> /input1/F2_O
- U2 pad 113: /hdmitx1/B5 -> /input1/F1_O
- U2 pad 114: /hdmitx1/B6 -> /input1/F0_O
- U2 pad 115: /hdmitx1/B7 -> /input1/R3_O
- U2 pad 119: /hdmitx1/G0 -> Net-(U2-Pad119)
- U2 pad 120: /fpga1/HDMITX_PCLK -> /input1/R2_O
- U2 pad 121: /hdmitx1/G1 -> /input1/R1_O
- U2 pad 125: /hdmitx1/G2 -> /input1/R0_O
- U2 pad 126: GND -> /input1/G3_O
- U2 pad 127: GND -> /input1/G2_O
- U2 pad 128: GND -> /input1/G1_O
- U2 pad 129: GND -> /input1/G0_O
- U2 pad 132: /hdmitx1/G3 -> /input1/B3_O
- U2 pad 133: /hdmitx1/G4 -> /input1/B2_O
- U2 pad 134: /hdmitx1/G5 -> /fpga1/VCCINT
- U2 pad 135: /hdmitx1/G6 -> /input1/B1_O
- U2 pad 136: /hdmitx1/G7 -> Net-(U2-Pad136)
- U2 pad 137: /fpga1/HDMITX_R0 -> /input1/B0_O
- U2 pad 141: /fpga1/HDMITX_R1 -> /fpga1/SDA
- U2 pad 142: /fpga1/HDMITX_R2 -> /fpga1/SCL
- U2 pad 143: /fpga1/HDMITX_R3 -> /input1/VOL+_O
- U2 pad 144: /fpga1/HDMITX_R4 -> /input1/VOL-_O
- U2 pad 22: GND -> /fpga1/BCKO
- U2 pad 23: GND -> /input1/CLK1
- U2 pad 24: GND -> /input1/CLK0
- U2 pad 25: GND -> /input1/PCLKx2
- U2 pad 28: Net-(U2-Pad28) -> /input1/HSYNC_O
- U2 pad 30: /fpga1/SDA -> GND
- U2 pad 31: /fpga1/SCL -> /fpga1/HDMITX_I2S_WS
- U2 pad 32: Net-(U2-Pad32) -> /input1/VSYNC_O
- U2 pad 33: Net-(U2-Pad33) -> /fpga1/HDMITX_I2S_BCK
- U2 pad 39: /input1/F3_O -> /fpga1/HDMITX_VSYNC
- U2 pad 42: /input1/F2_O -> /fpga1/HDMITX_HSYNC
- U2 pad 43: /input1/F1_O -> /hdmitx1/DE
- U2 pad 44: /input1/F0_O -> /hdmitx1/B0
- U2 pad 46: /input1/R3_O -> /fpga1/HDMITX_I2S_DATA
- U2 pad 49: /input1/R2_O -> /hdmitx1/B1
- U2 pad 50: /input1/R1_O -> /hdmitx1/B2
- U2 pad 51: /input1/R0_O -> /hdmitx1/B3
- U2 pad 55: /fpga1/I2S_BCK -> GND
- U2 pad 58: /fpga1/I2S_WS -> /hdmitx1/B4
- U2 pad 59: /fpga1/I2S_DATA -> /hdmitx1/B5
- U2 pad 60: /input1/VOL+_O -> /hdmitx1/B6
- U2 pad 61: /input1/VOL-_O -> /fpga1/VCCINT
- U2 pad 64: /input1/G3_O -> GND
- U2 pad 65: /input1/G2_O -> /fpga1/HDMITX_INT_N
- U2 pad 66: /input1/G1_O -> /hdmitx1/B7
- U2 pad 67: /input1/G0_O -> /hdmitx1/G0
- U2 pad 68: /input1/B3_O -> /fpga1/HDMITX_PCLK
- U2 pad 69: /input1/B2_O -> /hdmitx1/G1
- U2 pad 7: /fpga1/HDMITX_R5 -> Net-(U2-Pad7)
- U2 pad 71: /input1/B1_O -> /hdmitx1/G2
- U2 pad 72: /input1/B0_O -> /hdmitx1/G3
- U2 pad 76: Net-(U2-Pad76) -> /hdmitx1/G4
- U2 pad 77: Net-(U2-Pad77) -> /hdmitx1/G5
- U2 pad 83: Net-(U2-Pad83) -> /hdmitx1/G6
- U2 pad 85: /fpga1/HDMITX_RESET_N -> /hdmitx1/G7
- U2 pad 86: /fpga1/HDMITX_INT_N -> /fpga1/HDMITX_R0
- U2 pad 87: /fpga1/HDMITX_I2S_BCK -> /fpga1/HDMITX_R1
- U2 pad 88: /fpga1/CLK0 -> GND
- U2 pad 89: /input1/PCLKx2 -> GND
- U2 pad 90: /input1/VSYNC_O -> GND
- U2 pad 91: /input1/HSYNC_O -> GND
- U2 pad 98: /fpga1/HDMITX_I2S_WS -> /fpga1/HDMITX_R2
- U2 pad 99: /fpga1/HDMITX_I2S_DATA -> /fpga1/HDMITX_R3
- U6 pad 12: Net-(U6-Pad12) -> /input1/CLK1
- U6 pad 13: /fpga1/CLK0 -> /input1/CLK0
- U6 pad 20: /hdmitx1/DVDD3V3 -> /A33VDD
Routing:
- net /input1/VSYNC_O: track 13.1 -> 1.05 mm
- net /fpga1/TMS: track 0.00 -> 12.0 mm
- net GND: track 0.00 -> 10.5 mm
- net /input1/HSYNC_O: track 11.6 -> 1.06 mm
- net /hdmitx1/DVDD3V3: track 0.00 -> 9.48 mm
- net /input1/PCLKx2: track 13.5 -> 4.11 mm
- net /fpga1/TCK: track 0.00 -> 5.06 mm
- net /fpga1/CLK0: track 5.06 -> 0.00 mm
- net /hdmitx1/TXC+: track 11.1 -> 12.4 mm
- net /hdmitx1/TX1+: track 11.1 -> 12.4 mm
- net /hdmitx1/TX2-: track 11.1 -> 12.4 mm
- net /hdmitx1/TX0+: track 11.1 -> 12.4 mm
- net /hdmitx1/TX0-: track 11.1 -> 12.4 mm
- net /hdmitx1/TXC-: track 11.1 -> 12.4 mm
- net /hdmitx1/TX2+: track 11.1 -> 12.4 mm
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Other:
- board text added: "CPS2_digiAV v2.0"
- board text removed: "CPS2_digiAV_Surfboard v0.1"

Commit message: pcb: signal routing mostly done
Parts:
- removed C24: 10u, custom_components:SM0603_Capa_libcms
- added J7: GS2, Connectors:GS2, F.Cu at (78.6, 59.8)
- added R6: 10k, custom_components:SM0603_Resistor_libcms, F.Cu at (81.6, 59.7)
- C1, C14, C3, C5, C6, C7, C8, R20, R21, R22, R4: moved to F.Cu
- C15, C16, C17, C9: moved to B.Cu
- J1, J2: footprint Housings_DIP:DIP-10_W7.62mm_LongPads -> custom_components:HLE-105-02-G-DV-PE
- moved R24 75.0 mm to (34.3, 71.0), turned to 180 degrees
- moved R23 73.1 mm to (34.4, 69.3)
- moved R5 70.7 mm to (120.5, 30.0)
- moved R19 67.7 mm to (34.4, 72.7)
- moved C55 66.2 mm to (34.4, 67.6)
- moved U10 44.8 mm to (44.3, 69.5)
- moved C94 37.8 mm to (106.2, 92.4)
- moved U12 36.5 mm to (106.2, 88.7)
- moved C96 36.1 mm to (106.2, 84.7)
- moved C17 33.9 mm to (81.5, 51.7), turned to 90 degrees
- moved C91 33.4 mm to (113.3, 86.4)
- moved C8 33.1 mm to (72.0, 63.4), turned to 270 degrees
- moved U13 32.9 mm to (112.5, 82.3)
- moved C97 32.2 mm to (112.5, 78.3)
- moved C25 32.0 mm to (89.0, 68.7), turned to 270 degrees
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Connections:
- J1 pad 10: Net-(J1-Pad10) -> /input1/G3
- J1 pad 2: Net-(J1-Pad2) -> /input1/B0
- J1 pad 3: Net-(J1-Pad3) -> /input1/B1
- J1 pad 4: Net-(J1-Pad4) -> /input1/B2
- J1 pad 6: Net-(J1-Pad6) -> /input1/B3
- J1 pad 7: Net-(J1-Pad7) -> /input1/G0
- J1 pad 8: Net-(J1-Pad8) -> /input1/G1
- J1 pad 9: Net-(J1-Pad9) -> /input1/G2
- J2 pad 10: Net-(J2-Pad10) -> /input1/F3
- J2 pad 2: Net-(J2-Pad2) -> /input1/R0
- J2 pad 3: Net-(J2-Pad3) -> /input1/R1
- J2 pad 4: Net-(J2-Pad4) -> /input1/R2
- J2 pad 6: Net-(J2-Pad6) -> /input1/R3
- J2 pad 7: Net-(J2-Pad7) -> /input1/F0
- J2 pad 8: Net-(J2-Pad8) -> /input1/F1
- J2 pad 9: Net-(J2-Pad9) -> /input1/F2
- U11 pad 2: /input1/CLK1 -> /input1/CLK0
- U11 pad 9: GND -> /fpga1/ASRC_BYP
- U2 pad 111: /input1/F3_O -> /input1/R2_O
- U2 pad 112: /input1/F2_O -> /input1/R1_O
- U2 pad 113: /input1/F1_O -> /input1/R0_O
- U2 pad 114: /input1/F0_O -> /input1/F3_O
- U2 pad 115: /input1/R3_O -> /input1/F2_O
- U2 pad 120: /input1/R2_O -> /input1/F1_O
- U2 pad 121: /input1/R1_O -> /input1/F0_O
- U2 pad 125: /input1/R0_O -> /input1/R3_O
- U2 pad 126: /input1/G3_O -> /input1/B2_O
- U2 pad 127: /input1/G2_O -> /input1/B1_O
- U2 pad 128: /input1/G1_O -> /input1/B0_O
- U2 pad 129: /input1/G0_O -> /input1/B3_O
- U2 pad 132: /input1/B3_O -> /input1/G0_O
- U2 pad 133: /input1/B2_O -> /input1/G1_O
- U2 pad 135: /input1/B1_O -> /input1/G2_O
- U2 pad 137: /input1/B0_O -> /input1/G3_O
- U2 pad 23: /input1/CLK1 -> /input1/CLK0
- U2 pad 24: /input1/CLK0 -> /input1/CLK1
- U2 pad 28: /input1/HSYNC_O -> /input1/VSYNC_O
- U2 pad 31: /fpga1/HDMITX_I2S_WS -> /input1/HSYNC_O
- U2 pad 32: /input1/VSYNC_O -> /fpga1/HDMITX_I2S_WS
- U3 pad 11: /input1/R0_O -> /input1/R3_O
- U3 pad 12: /input1/R1_O -> /input1/F0_O
- U3 pad 13: /input1/R2_O -> /input1/F1_O
- U3 pad 14: /input1/R3_O -> /input1/F2_O
- U3 pad 15: /input1/F0_O -> /input1/F3_O
- U3 pad 16: /input1/F1_O -> /input1/R0_O
- U3 pad 17: /input1/F2_O -> /input1/R1_O
- U3 pad 18: /input1/F3_O -> /input1/R2_O
- U3 pad 2: Net-(J2-Pad10) -> /input1/R2
- U3 pad 3: Net-(J2-Pad9) -> /input1/R1
- U3 pad 4: Net-(J2-Pad8) -> /input1/R0
- U3 pad 5: Net-(J2-Pad7) -> /input1/F3
- U3 pad 6: Net-(J2-Pad6) -> /input1/F2
- U3 pad 7: Net-(J2-Pad4) -> /input1/F1
- U3 pad 8: Net-(J2-Pad3) -> /input1/F0
- U3 pad 9: Net-(J2-Pad2) -> /input1/R3
- U4 pad 11: /input1/B0_O -> /input1/G3_O
- U4 pad 12: /input1/B1_O -> /input1/G2_O
- U4 pad 13: /input1/B2_O -> /input1/G1_O
- U4 pad 14: /input1/B3_O -> /input1/G0_O
- U4 pad 15: /input1/G0_O -> /input1/B3_O
- U4 pad 16: /input1/G1_O -> /input1/B0_O
- U4 pad 17: /input1/G2_O -> /input1/B1_O
- U4 pad 18: /input1/G3_O -> /input1/B2_O
- U4 pad 2: Net-(J1-Pad10) -> /input1/B2
- U4 pad 3: Net-(J1-Pad9) -> /input1/B1
- U4 pad 4: Net-(J1-Pad8) -> /input1/B0
- U4 pad 5: Net-(J1-Pad7) -> /input1/B3
- U4 pad 6: Net-(J1-Pad6) -> /input1/G0
- U4 pad 7: Net-(J1-Pad4) -> /input1/G1
- U4 pad 8: Net-(J1-Pad3) -> /input1/G2
- U4 pad 9: Net-(J1-Pad2) -> /input1/G3
- U5 pad 14: /input1/VOL-_O -> /fpga1/I2S_WS
- U5 pad 15: /input1/VOL+_O -> /fpga1/I2S_BCK
- U5 pad 17: /fpga1/I2S_WS -> /input1/VOL-_O
- U5 pad 18: /fpga1/I2S_BCK -> /input1/VOL+_O
- U5 pad 7: Net-(U5-Pad7) -> GND
- U5 pad 8: Net-(U5-Pad8) -> GND
- U5 pad 9: Net-(U5-Pad9) -> GND
- W2 pad 1: Net-(U5-Pad2) -> Net-(U5-Pad5)
- W3 pad 1: Net-(U5-Pad3) -> Net-(U5-Pad6)
- W5 pad 1: Net-(U5-Pad5) -> Net-(U5-Pad2)
- W6 pad 1: Net-(U5-Pad6) -> Net-(U5-Pad3)
Routing:
- net /input1/R2: track 0.00 -> 42.5 mm
- net /fpga1/HDMITX_R7: track 0.00 -> 41.8 mm
- net /fpga1/HDMITX_R6: track 0.00 -> 39.5 mm
- net /input1/R1: track 0.00 -> 38.9 mm
- net /fpga1/HDMITX_R5: track 0.00 -> 37.8 mm
- net /fpga1/HDMITX_R4: track 0.00 -> 36.5 mm
- net /input1/R0: track 0.00 -> 35.3 mm
- net /fpga1/HDMITX_R3: track 0.00 -> 35.2 mm
- net /hdmitx1/DDCSDA: track 0.00 -> 34.4 mm
- net /fpga1/HDMITX_R2: track 0.00 -> 33.8 mm
- net /fpga1/HDMITX_I2S_WS: track 0.00 -> 29.6 mm
- net /input1/R3: track 0.00 -> 29.3 mm
- net /fpga1/HDMITX_R1: track 0.00 -> 27.7 mm
- net /input1/F0: track 0.00 -> 27.4 mm
- net /fpga1/HDMITX_I2S_BCK: track 0.00 -> 26.9 mm
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Other:
- board size 103.4 x 48.7 mm -> 103.4 x 43.5 mm

Commit message: finalize rev. 2.0 pcb
Parts:
- removed C110: 10u, custom_components:SM0603_Capa_libcms
- removed C2, C4, C52, C88, C90: 1u, custom_components:SM0603_Capa_libcms
- removed U16: TLV70018, custom_components:SOT-23-5_Handsoldering
- removed U8: TLV70033, custom_components:SOT-23-5_Handsoldering
- C16, C55, R19, R23, R24: moved to F.Cu
- C18, C19, C20, C21, C22, C46: moved to B.Cu
- moved C20 42.6 mm to (79.3, 43.0), turned to 180 degrees
- moved C22 42.0 mm to (101.9, 41.5)
- moved R24 41.6 mm to (47.4, 31.4)
- moved R19 40.6 mm to (43.2, 33.1)
- moved C18 38.7 mm to (101.9, 46.7)
- moved C21 38.4 mm to (101.9, 43.2)
- moved C55 37.2 mm to (43.2, 31.4)
- moved C19 36.4 mm to (79.3, 48.6), turned to 180 degrees
- moved C12 31.1 mm to (119.3, 51.0), turned to 270 degrees
- moved FB2 31.0 mm to (117.6, 51.0), turned to 90 degrees
- moved U10 30.4 mm to (44.6, 39.1), turned to 90 degrees
- moved C46 30.3 mm to (99.5, 56.6), turned to 270 degrees
- moved C69 29.6 mm to (118.9, 46.0), turned to 270 degrees
- moved C64 27.9 mm to (98.4, 34.0), turned to 90 degrees
- moved C61 27.6 mm to (83.1, 34.0), turned to 90 degrees
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Connections:
- net Net-(C10-Pad1) renamed /hdmitx1/DVDD1V8_FILT_DVDD
- net Net-(C12-Pad1) renamed /hdmitx1/DVDD1V8_FILT_PVDD
- net Net-(C13-Pad1) renamed /hdmitx1/DVDD1V8_FILT_AVDD
- C11 pad 1: Net-(C11-Pad1) -> /hdmitx1/DVDD3V3_FILT_DVDD_3V
- C16 pad 2: /A33VDD -> /hdmitx1/DVDD3V3
- C5 pad 1: /input1/5V -> /5V
- C82 pad 1: Net-(C11-Pad1) -> /hdmitx1/DVDD3V3_FILT_DVDD_3V
- C85 pad 1: /hdmitx1/AVDD1V8 -> /hdmitx1/DVDD1V8
- C86 pad 1: /hdmitx1/AVDD1V8 -> /hdmitx1/DVDD1V8
- D1 pad 1: /input1/5V -> /5V
- D2 pad 8: Net-(D2-Pad8) -> GND
- D3 pad 8: Net-(D3-Pad8) -> GND
- FB1 pad 1: /hdmitx1/AVDD1V8 -> /hdmitx1/DVDD1V8
- FB2 pad 1: /hdmitx1/AVDD1V8 -> /hdmitx1/DVDD1V8
- FB4 pad 1: Net-(C11-Pad1) -> /hdmitx1/DVDD3V3_FILT_DVDD_3V
- R5 pad 1: /hdmitx1/DVDD3V3 -> /hdmitx1/DVDD3V3_FILT_DVDD_3V
- U1 pad 29: Net-(C11-Pad1) -> /hdmitx1/DVDD3V3_FILT_DVDD_3V
- U2 pad 10: /fpga1/SDOUT -> /fpga1/LRCKO
- U2 pad 11: /fpga1/LRCKO -> /fpga1/SDOUT
- U6 pad 20: /A33VDD -> /hdmitx1/DVDD3V3
- W1 pad 1: /input1/5V -> /5V
Routing:
- net GND: track 4.82 -> 1189.3 mm, vias 0 -> 193
- net /hdmitx1/DVDD3V3: track 0.12 -> 463.3 mm, vias 0 -> 27
- net /fpga1/VCCA: track 4.96 -> 165.7 mm, vias 0 -> 8
- net /fpga1/VCCINT: track 0.00 -> 148.1 mm, vias 0 -> 14
- net /fpga1/SDA: track 3.48 -> 120.1 mm, vias 0 -> 4
- net /fpga1/SCL: track 5.57 -> 114.3 mm, vias 0 -> 4
- net /fpga1/VCCD_PLL: track 0.00 -> 102.7 mm, vias 0 -> 9
- net /fpga1/DCLK: track 0.00 -> 63.2 mm, vias 0 -> 2
- net /fpga1/ASDO: track 0.00 -> 59.2 mm, vias 0 -> 2
- net /fpga1/nCSO: track 0.00 -> 59.0 mm, vias 0 -> 2
- net /fpga1/TDI: track 8.43 -> 65.7 mm, vias 0 -> 2
- net /5V: track 0.00 -> 55.3 mm, vias 0 -> 2
- net /fpga1/DATA0: track 0.00 -> 55.3 mm, vias 0 -> 2
- net /fpga1/TMS: track 7.92 -> 58.3 mm, vias 0 -> 1
- net /fpga1/TDO: track 0.00 -> 44.5 mm, vias 0 -> 1
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- added copper zone on B.Cu, net GND
- added copper zone on F.Cu, net GND
Other:
- board size 103.4 x 43.5 mm -> 103.9 x 43.5 mm

Commit message: update PCB to v2.1
Parts:
- added C2: 0.1u, custom_components:SM0603_Capa_libcms, F.Cu at (56.1, 61.1)
- added D4: ZHCS400TA, custom_components:SOD-323_Handsoldering, B.Cu at (129.8, 56.3)
- added R7: 10k, custom_components:SM0603_Resistor_libcms, B.Cu at (44.8, 68.0)
- added R8: 10k, custom_components:SM0603_Resistor_libcms, B.Cu at (46.5, 68.0)
- added SW1: TL2243, custom_components:TL2243, F.Cu at (45.7, 70.5)
- added U16: SN74LVC2G17, custom_components:SOT-23-6_Handsoldering, F.Cu at (102.0, 64.7)
- added U8: SN74LVC2G17, custom_components:SOT-23-6_Handsoldering, F.Cu at (55.3, 64.9)
- added W14: GND, custom_components:SMD_PAD, F.Cu at (61.9, 70.5)
- added W15: C1, custom_components:SMD_PAD, F.Cu at (97.3, 70.5)
- U9: value SN74LVC3G17 -> SN74LVC2G17; footprint custom_components:SSOP-8_3x3mm_Pitch0.65mm -> custom_components:SOT-23-6_Handsoldering
- W11: value HSYNC -> HS
- W12: value VSYNC -> VS
- W13: value PCLKx2 -> C2
- W2: value I2S_BCK -> BCK
- W3: value I2S_WS -> WS
- W4: value I2S_DATA -> DAT
- W5: value btn_vol+ -> vol+
- W6: value btn_vol- -> vol-
- moved W12 7.50 mm to (103.0, 70.5)
- moved W11 5.75 mm to (105.0, 70.5)
- moved R6 4.11 mm to (77.5, 59.7)
- moved W13 3.90 mm to (99.2, 70.4)
- moved W4 3.84 mm to (59.9, 70.4)
- moved C14 2.73 mm to (104.7, 61.3)
- moved W7 1.99 mm to (95.4, 70.5)
- moved W2 1.98 mm to (56.0, 70.4)
- moved W8 1.96 mm to (106.9, 70.4)
- moved W3 1.94 mm to (58.0, 70.4)
- moved J7 1.87 mm to (80.5, 59.7)
- moved U9 1.72 mm to (98.3, 64.7)
- moved W5 0.73 mm to (51.5, 70.4)
- moved W6 0.73 mm to (53.5, 70.4)
- moved W10 0.14 mm to (101.1, 70.4)
Connections:
- net /input1/CLK1 renamed /fpga1/PCLK_SI
- F2 pad 1: /5V -> Net-(D4-Pad1)
- J7 pad 1: /hdmitx1/DVDD3V3 -> /fpga1/LGRP
- J7 pad 2: /fpga1/ASRC_BYP -> GND
- R6 pad 1: GND -> /fpga1/LGRP
- R6 pad 2: /fpga1/ASRC_BYP -> /hdmitx1/DVDD3V3
- U11 pad 1: /hdmitx1/DVDD3V3 -> /fpga1/LGRP
- U11 pad 2: /input1/CLK0 -> /fpga1/MCLK_SI
- U11 pad 9: /fpga1/ASRC_BYP -> GND
- U2 pad 23: /input1/CLK0 -> /fpga1/MCLK_SI
- U2 pad 25: /input1/PCLKx2 -> /input1/PCLK
- U5 pad 13: Net-(U5-Pad13) -> /fpga1/I2S_WS
- U5 pad 14: /fpga1/I2S_WS -> Net-(U5-Pad14)
- U5 pad 15: /fpga1/I2S_BCK -> Net-(U5-Pad15)
- U5 pad 5: Net-(U5-Pad5) -> GND
- U5 pad 6: Net-(U5-Pad6) -> GND
- U5 pad 7: GND -> Net-(U5-Pad7)
- U6 pad 13: /input1/CLK0 -> Net-(U6-Pad13)
- U6 pad 16: Net-(U6-Pad16) -> /fpga1/MCLK_SI
- U6 pad 6: /input1/PCLKx2 -> Net-(U6-Pad6)
- U9 pad 2: /input1/PCLKx2 -> GND
- U9 pad 4: GND -> /input1/PCLK
- U9 pad 5: /input1/VSYNC_O -> /hdmitx1/DVDD3V3
- U9 pad 6: Net-(U9-Pad6) -> Net-(U6-Pad6)
- W11 pad 1: Net-(U9-Pad1) -> Net-(U16-Pad3)
- W12 pad 1: Net-(U9-Pad3) -> Net-(U16-Pad1)
- W13 pad 1: Net-(U9-Pad6) -> Net-(U9-Pad3)
- W2 pad 1: Net-(U5-Pad5) -> Net-(U8-Pad3)
- W3 pad 1: Net-(U5-Pad6) -> Net-(U5-Pad7)
Routing:
- net GND: track 1189.3 -> 1280.2 mm, vias 193 -> 207
- net /input1/CLK0: track 22.1 -> 0.00 mm
- net /fpga1/MCLK_SI: track 0.00 -> 21.5 mm
- net /hdmitx1/DVDD3V3: track 463.3 -> 483.8 mm, vias 27 -> 30
- net /fpga1/I2S_BCK: track 11.7 -> 30.9 mm, vias 0 -> 2
- net /input1/PCLKx2: track 12.9 -> 0.00 mm
- net /fpga1/ASRC_BYP: track 12.2 -> 0.00 mm, vias 2 -> 0
- net Net-(R8-Pad2): track 13.9 -> 24.7 mm, vias 0 -> 2
- net Net-(R7-Pad2): track 16.1 -> 26.8 mm, vias 0 -> 2
- net Net-(U5-Pad7): track 0.00 -> 10.0 mm, vias 0 -> 2
- net /input1/PCLK: track 0.00 -> 9.70 mm
- net /5V: track 55.3 -> 45.7 mm, vias 2 -> 1
- net Net-(U5-Pad5): track 9.23 -> 0.00 mm
- net Net-(U9-Pad6): track 6.97 -> 0.00 mm
- net Net-(D4-Pad1): track 0.00 -> 6.56 mm, vias 0 -> 1
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Other:
- outline, holes or cut-outs redrawn
- rule pad_to_mask_clearance: 0 -> 0.0508
- board text added: "CPS2_digiAV v2.1"
- board text removed: "CPS2_digiAV v2.0"
